Commit message: moveit working

File: ipa_seminar_application/ipa_seminar_application/helper/ur.urdf.xacro (robot description, xacro)
@@ -4,13 +4,10 @@
        xmlns:interface="http://playerstage.sourceforge.net/gazebo/xmlschema/#interface"
        xmlns:xacro="http://playerstage.sourceforge.net/gazebo/xmlschema/#interface"
-       name="ur" >
+       name="ur10" >
   <!-- common stuff -->
-  <include filename="$(find cob_description)/urdf/common.xacro" />
-  <include filename="$(find cob_description)/urdf/materials.urdf.xacro" />
-  <include filename="$(find cob_description)/gazebo/gazebo.urdf.xacro" />
-  <!-- calibration -->
-  <!--include filename="$(find ipa_seminar_application)/helper/calibration_ur.urdf.xacro" /-->
-  <!-- ur -->
-  <include filename="$(find ur_description)/urdf/ur5.urdf.xacro" />
+  <include filename="$(find ur_description)/urdf/gazebo.urdf.xacro" />
+  <!-- ur10 -->
+  <!--include filename="$(find ur_description)/urdf/ur10.urdf.xacro" /-->
+  <include filename="$(find raw_description)/urdf/ur_arm/ur10_arm.urdf.xacro" />
   <!-- foot for arm -->
 	<link name="base_link">
@@ -23,18 +20,18 @@
 		   <origin xyz="0 0 0.5" rpy="0 0 0" />
 		   <geometry>
-			  <box size="1 1 1"/>
+			  <box size="2 2 1"/>
 		   </geometry>
-		   <material name="Schunk/DarkGrey" />
+		   <material name="White" />
 		</visual>
 		<collision>
 		   <origin xyz="0 0 0.5" rpy="0 0 0" />
 		   <geometry>
-			  <box size="1 1 1"/>
+			  <box size="2 2 1"/>
 		   </geometry>
 		</collision>
 	</link>
   <!-- arm -->
-  <xacro:ur5_robot prefix="arm_" >
-    <origin xyz="0 0 1" rpy="0 0 0" />
-  </xacro:ur5_robot>
+  <xacro:cob_ur10 name="arm" parent="base_link">
+      <origin xyz="0 0 1" rpy="0 0 0" />
+  </xacro:cob_ur10>
 </robot>
