Commit message: add gripper

File: ipa_seminar_application/ipa_seminar_application_bringup/urdf/ur.urdf.xacro (robot description, xacro)
@@ -7,4 +7,5 @@
   <!-- common stuff -->
   <include filename="$(find ur_description)/urdf/gazebo.urdf.xacro" />
+  <include filename="$(find schunk_description)/urdf/pg70/pg70.urdf.xacro" />
   <!-- ur10 -->
   <!--include filename="$(find ur_description)/urdf/ur10.urdf.xacro" /-->
@@ -35,3 +36,7 @@
       <origin xyz="0 0 1" rpy="0 0 0" />
   </xacro:cob_ur10>
+  <!-- gripper -->
+  <xacro:schunk_pg70 name="gripper" parent="arm_ee_link">
+      <origin xyz="0 0 0" rpy="0 0 0" />
+  </xacro:schunk_pg70>
 </robot>

Commit message: fix gripper orientation

File: ipa_seminar_application/ipa_seminar_application_bringup/urdf/ur.urdf.xacro (robot description, xacro)
@@ -38,5 +38,5 @@
   <!-- gripper -->
   <xacro:schunk_pg70 name="gripper" parent="arm_ee_link">
-      <origin xyz="0 0 0" rpy="0 0 0" />
+      <origin xyz="0 0 0" rpy="0 1.5708 0" />
   </xacro:schunk_pg70>
 </robot>
