Commit message: urdfs for ur, lbr and lwa4d

File: ipa_seminar_application/ipa_seminar_application_bringup/urdf/lbr.urdf.xacro (robot description, xacro)
@@ -9,6 +9,5 @@
   <include filename="$(find cob_description)/urdf/materials.urdf.xacro" />
   <include filename="$(find cob_description)/gazebo/gazebo.urdf.xacro" />
-  <!-- calibration -->
-  <!--include filename="$(find ipa_seminar_application_bringup)/helper/calibration_lbr.urdf.xacro" /-->
+  <include filename="$(find schunk_description)/urdf/pg70/pg70.urdf.xacro" />
   <!-- lbr -->
   <include filename="$(find cob_description)/urdf/lbr/lbr.urdf.xacro" />
@@ -23,12 +22,12 @@
 		   <origin xyz="0 0 0.5" rpy="0 0 0" />
 		   <geometry>
-			  <box size="1 1 1"/>
+			  <box size="2 2 1"/>
 		   </geometry>
-		   <material name="Schunk/DarkGrey" />
+		   <material name="IPA/LightGrey" />
 		</visual>
 		<collision>
 		   <origin xyz="0 0 0.5" rpy="0 0 0" />
 		   <geometry>
-			  <box size="1 1 1"/>
+			  <box size="2 2 1"/>
 		   </geometry>
 		</collision>
@@ -38,3 +37,7 @@
     <origin xyz="0 0 1" rpy="0 0 0" />
   </xacro:cob_lbr>
+  <!-- gripper -->
+  <xacro:schunk_pg70 name="gripper" parent="arm_7_link">
+      <origin xyz="0 0 0.02" rpy="0 0 0" />
+  </xacro:schunk_pg70>
 </robot>

File: ipa_seminar_application/ipa_seminar_application_bringup/urdf/lwa4d.urdf.xacro (robot description, xacro)
@@ -9,6 +9,7 @@
   <include filename="$(find cob_description)/urdf/materials.urdf.xacro" />
   <include filename="$(find cob_description)/gazebo/gazebo.urdf.xacro" />
+  <include filename="$(find schunk_description)/urdf/pg70/pg70.urdf.xacro" />
   <!-- calibration -->
-  <include filename="$(find ipa_seminar_application_bringup)/helper/calibration_lwa4d.urdf.xacro" />
+  <include filename="$(find ipa_seminar_application_bringup)/urdf/calibration_lwa4d.urdf.xacro" />
   <!-- lwa4d -->
   <include filename="$(find schunk_description)/urdf/lwa4d/lwa4d.urdf.xacro" />
@@ -23,12 +24,12 @@
 		   <origin xyz="0 0 0.5" rpy="0 0 0" />
 		   <geometry>
-			  <box size="1 1 1"/>
+			  <box size="2 2 1"/>
 		   </geometry>
-		   <material name="Schunk/DarkGrey" />
+		   <material name="IPA/LightGrey" />
 		</visual>
 		<collision>
 		   <origin xyz="0 0 0.5" rpy="0 0 0" />
 		   <geometry>
-			  <box size="1 1 1"/>
+			  <box size="2 2 1"/>
 		   </geometry>
 		</collision>
@@ -36,5 +37,9 @@
   <!-- arm -->
   <xacro:schunk_lwa4d name="arm" parent="base_link">
-    <origin xyz="0 0 2" rpy="3.1415926 0 0" />
+    <origin xyz="0 0 1" rpy="3.1415926 0 0" />
   </xacro:schunk_lwa4d>
+  <!-- gripper -->
+  <xacro:schunk_pg70 name="gripper" parent="arm_7_link">
+      <origin xyz="0 0 0" rpy="3.14 0 0" />
+  </xacro:schunk_pg70>
 </robot>

File: ipa_seminar_application/ipa_seminar_application_bringup/urdf/ur.urdf.xacro (robot description, xacro)
@@ -7,7 +7,9 @@
   <!-- common stuff -->
   <include filename="$(find ur_description)/urdf/gazebo.urdf.xacro" />
+  <include filename="$(find cob_description)/urdf/common.xacro" />
+  <include filename="$(find cob_description)/urdf/materials.urdf.xacro" />
+  <include filename="$(find cob_description)/gazebo/gazebo.urdf.xacro" />
   <include filename="$(find schunk_description)/urdf/pg70/pg70.urdf.xacro" />
   <!-- ur10 -->
-  <!--include filename="$(find ur_description)/urdf/ur10.urdf.xacro" /-->
   <include filename="$(find raw_description)/urdf/ur_arm/ur10_arm.urdf.xacro" />
   <!-- foot for arm -->
@@ -23,5 +25,5 @@
 			  <box size="2 2 1"/>
 		   </geometry>
-		   <material name="White" />
+		   <material name="IPA/LightGrey" />
 		</visual>
 		<collision>
@@ -34,5 +36,5 @@
   <!-- arm -->
   <xacro:cob_ur10 name="arm" parent="base_link">
-      <origin xyz="0 0 1" rpy="0 0 0" />
+    <origin xyz="0 0 1" rpy="0 0 0" />
   </xacro:cob_ur10>
   <!-- gripper -->

Commit message: fix simulation with ur

File: ipa_seminar_application/ipa_seminar_application_bringup/urdf/lbr.urdf.xacro (robot description, xacro)
@@ -1,36 +1,33 @@
 <?xml version="1.0"?>
-<robot xmlns:sensor="http://playerstage.sourceforge.net/gazebo/xmlschema/#sensor"
-       xmlns:controller="http://playerstage.sourceforge.net/gazebo/xmlschema/#controller"
-       xmlns:interface="http://playerstage.sourceforge.net/gazebo/xmlschema/#interface"
-       xmlns:xacro="http://playerstage.sourceforge.net/gazebo/xmlschema/#interface"
+<robot xmlns:xacro="http://www.ros.org/wiki/xacro"
        name="lbr" >
   <!-- common stuff -->
-  <include filename="$(find cob_description)/urdf/common.xacro" />
-  <include filename="$(find cob_description)/urdf/materials.urdf.xacro" />
-  <include filename="$(find cob_description)/gazebo/gazebo.urdf.xacro" />
-  <include filename="$(find schunk_description)/urdf/pg70/pg70.urdf.xacro" />
+  <xacro:include filename="$(find cob_description)/urdf/common.xacro" />
+  <xacro:include filename="$(find cob_description)/urdf/materials.urdf.xacro" />
+  <xacro:include filename="$(find schunk_description)/urdf/pg70/pg70.urdf.xacro" />
   <!-- lbr -->
-  <include filename="$(find cob_description)/urdf/lbr/lbr.urdf.xacro" />
+  <xacro:include filename="$(find cob_description)/urdf/lbr/lbr.urdf.xacro" />
+  <link name="world"/>
+  <joint name="world_joint" type="fixed">
+    <origin xyz="0 0 0.5" rpy="0 0 0" />
+    <parent link="world"/>
+    <child link="base_link"/>
+  </joint>
   <!-- foot for arm -->
-	<link name="base_link">
-		<inertial>
-		   <origin xyz="0 0 -10" rpy="0 0 0"/>
-		   <mass value="1000.0"/>
-		   <inertia ixx="100.0"  ixy="0"  ixz="0" iyy="100.0" iyz="0" izz="100.0" />
-		</inertial>
-		<visual>
-		   <origin xyz="0 0 0.5" rpy="0 0 0" />
-		   <geometry>
-			  <box size="2 2 1"/>
-		   </geometry>
-		   <material name="IPA/LightGrey" />
-		</visual>
-		<collision>
-		   <origin xyz="0 0 0.5" rpy="0 0 0" />
-		   <geometry>
-			  <box size="2 2 1"/>
-		   </geometry>
-		</collision>
-	</link>
+  <link name="base_link">
+	<visual>
+	  <origin xyz="0 0 0.5" rpy="0 0 0" />
+	  <geometry>
+		<box size="2 2 1"/>
+	  </geometry>
+	  <material name="IPA/LightGrey" />
+	</visual>
+	<collision>
+	  <origin xyz="0 0 0.5" rpy="0 0 0" />
+	  <geometry>
+		<box size="2 2 1"/>
+	  </geometry>
+	</collision>
+  </link>
   <!-- arm -->
   <xacro:cob_lbr name="arm" parent="base_link">
@@ -41,3 +38,9 @@
       <origin xyz="0 0 0.02" rpy="0 0 0" />
   </xacro:schunk_pg70>
+  <gazebo>
+    <plugin name="ros_control" filename="libgazebo_ros_control.so">
+      <!--robotNamespace>/</robotNamespace-->
+      <!--robotSimType>gazebo_ros_control/DefaultRobotHWSim</robotSimType-->
+    </plugin>
+  </gazebo>
 </robot>

File: ipa_seminar_application/ipa_seminar_application_bringup/urdf/lwa4d.urdf.xacro (robot description, xacro)
@@ -1,38 +1,33 @@
 <?xml version="1.0"?>
-<robot xmlns:sensor="http://playerstage.sourceforge.net/gazebo/xmlschema/#sensor"
-       xmlns:controller="http://playerstage.sourceforge.net/gazebo/xmlschema/#controller"
-       xmlns:interface="http://playerstage.sourceforge.net/gazebo/xmlschema/#interface"
-       xmlns:xacro="http://playerstage.sourceforge.net/gazebo/xmlschema/#interface"
+<robot xmlns:xacro="http://www.ros.org/wiki/xacro"
        name="lwa4d" >
   <!-- common stuff -->
-  <include filename="$(find cob_description)/urdf/common.xacro" />
-  <include filename="$(find cob_description)/urdf/materials.urdf.xacro" />
-  <include filename="$(find cob_description)/gazebo/gazebo.urdf.xacro" />
-  <include filename="$(find schunk_description)/urdf/pg70/pg70.urdf.xacro" />
-  <!-- calibration -->
-  <include filename="$(find ipa_seminar_application_bringup)/urdf/calibration_lwa4d.urdf.xacro" />
+  <xacro:include filename="$(find cob_description)/urdf/common.xacro" />
+  <xacro:include filename="$(find cob_description)/urdf/materials.urdf.xacro" />
+  <xacro:include filename="$(find schunk_description)/urdf/pg70/pg70.urdf.xacro" />
   <!-- lwa4d -->
-  <include filename="$(find schunk_description)/urdf/lwa4d/lwa4d.urdf.xacro" />
+  <xacro:include filename="$(find schunk_description)/urdf/lwa4d/lwa4d.urdf.xacro" />
+  <link name="world"/>
+  <joint name="world_joint" type="fixed">
+    <origin xyz="0 0 0.5" rpy="0 0 0" />
+    <parent link="world"/>
+    <child link="base_link"/>
+  </joint>
   <!-- foot for arm -->
-	<link name="base_link">
-		<inertial>
-		   <origin xyz="0 0 -10" rpy="0 0 0"/>
-		   <mass value="1000.0"/>
-		   <inertia ixx="100.0"  ixy="0"  ixz="0" iyy="100.0" iyz="0" izz="100.0" />
-		</inertial>
-		<visual>
-		   <origin xyz="0 0 0.5" rpy="0 0 0" />
-		   <geometry>
-			  <box size="2 2 1"/>
-		   </geometry>
-		   <material name="IPA/LightGrey" />
-		</visual>
-		<collision>
-		   <origin xyz="0 0 0.5" rpy="0 0 0" />
-		   <geometry>
-			  <box size="2 2 1"/>
-		   </geometry>
-		</collision>
-	</link>
+  <link name="base_link">
+	<visual>
+	  <origin xyz="0 0 0.5" rpy="0 0 0" />
+	  <geometry>
+		<box size="2 2 1"/>
+	  </geometry>
+	  <material name="IPA/LightGrey" />
+	</visual>
+	<collision>
+	  <origin xyz="0 0 0.5" rpy="0 0 0" />
+	  <geometry>
+		<box size="2 2 1"/>
+	  </geometry>
+	</collision>
+  </link>
   <!-- arm -->
   <xacro:schunk_lwa4d name="arm" parent="base_link">
@@ -43,3 +38,9 @@
       <origin xyz="0 0 0" rpy="0 0 0" />
   </xacro:schunk_pg70>
+  <gazebo>
+    <plugin name="ros_control" filename="libgazebo_ros_control.so">
+      <!--robotNamespace>/</robotNamespace-->
+      <!--robotSimType>gazebo_ros_control/DefaultRobotHWSim</robotSimType-->
+    </plugin>
+  </gazebo>
 </robot>

File: ipa_seminar_application/ipa_seminar_application_bringup/urdf/ur.urdf.xacro (robot description, xacro)
@@ -1,44 +1,46 @@
 <?xml version="1.0"?>
-<robot xmlns:sensor="http://playerstage.sourceforge.net/gazebo/xmlschema/#sensor"
-       xmlns:controller="http://playerstage.sourceforge.net/gazebo/xmlschema/#controller"
-       xmlns:interface="http://playerstage.sourceforge.net/gazebo/xmlschema/#interface"
-       xmlns:xacro="http://playerstage.sourceforge.net/gazebo/xmlschema/#interface"
+<robot xmlns:xacro="http://www.ros.org/wiki/xacro"
        name="ur10" >
   <!-- common stuff -->
-  <include filename="$(find ur_description)/urdf/gazebo.urdf.xacro" />
-  <include filename="$(find cob_description)/urdf/common.xacro" />
-  <include filename="$(find cob_description)/urdf/materials.urdf.xacro" />
-  <include filename="$(find cob_description)/gazebo/gazebo.urdf.xacro" />
-  <include filename="$(find schunk_description)/urdf/pg70/pg70.urdf.xacro" />
+  <xacro:include filename="$(find cob_description)/urdf/common.xacro" />
+  <xacro:include filename="$(find cob_description)/urdf/materials.urdf.xacro" />
+  <xacro:include filename="$(find schunk_description)/urdf/pg70/pg70.urdf.xacro" />
   <!-- ur10 -->
-  <include filename="$(find raw_description)/urdf/ur_arm/ur10_arm.urdf.xacro" />
+  <xacro:include filename="$(find cob_description)/urdf/ur_arm/ur10_arm.urdf.xacro" />
+  <link name="world"/>
+  <joint name="world_joint" type="fixed">
+    <origin xyz="0 0 0.5" rpy="0 0 0" />
+    <parent link="world"/>
+    <child link="base_link"/>
+  </joint>
   <!-- foot for arm -->
-	<link name="base_link">
-		<inertial>
-		   <origin xyz="0 0 -10" rpy="0 0 0"/>
-		   <mass value="1000.0"/>
-		   <inertia ixx="100.0"  ixy="0"  ixz="0" iyy="100.0" iyz="0" izz="100.0" />
-		</inertial>
-		<visual>
-		   <origin xyz="0 0 0.5" rpy="0 0 0" />
-		   <geometry>
-			  <box size="2 2 1"/>
-		   </geometry>
-		   <material name="IPA/LightGrey" />
-		</visual>
-		<collision>
-		   <origin xyz="0 0 0.5" rpy="0 0 0" />
-		   <geometry>
-			  <box size="2 2 1"/>
-		   </geometry>
-		</collision>
-	</link>
+  <link name="base_link">
+	<visual>
+	  <origin xyz="0 0 0.5" rpy="0 0 0" />
+	  <geometry>
+		<box size="2 2 1"/>
+	  </geometry>
+	  <material name="IPA/LightGrey" />
+	</visual>
+	<collision>
+	  <origin xyz="0 0 0.5" rpy="0 0 0" />
+	  <geometry>
+		<box size="2 2 1"/>
+	  </geometry>
+	</collision>
+  </link>
   <!-- arm -->
-  <xacro:cob_ur10 name="arm" parent="base_link">
+  <xacro:ur10 name="arm" parent="base_link">
     <origin xyz="0 0 1" rpy="0 0 0.40" />
-  </xacro:cob_ur10>
+  </xacro:ur10>
   <!-- gripper -->
   <xacro:schunk_pg70 name="gripper" parent="arm_ee_link">
       <origin xyz="0 0 0" rpy="0 1.5708 0" />
   </xacro:schunk_pg70>
+  <gazebo>
+    <plugin name="ros_control" filename="libgazebo_ros_control.so">
+      <!--robotNamespace>/</robotNamespace-->
+      <!--robotSimType>gazebo_ros_control/DefaultRobotHWSim</robotSimType-->
+    </plugin>
+  </gazebo>
 </robot>
